Commit message: 09/04

File: worlds/restaurant.urdf (robot description, URDF)
Before this commit: robot cube.urdf, 1 links, 0 joints
Links:
- link baseLink: geometry collision mesh filename=/home/georgiablanco/Downloads/4vi5shao064g-room/furniture_o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 scale=1 1 1; visual mesh filename=/home/georgiablanco/Downloads/4vi5shao064g-room/furniture_o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 scale=1 1 1

File: worlds/samurai_tables.urdf (robot description, URDF)
Before this commit: robot cube.urdf, 1 links, 0 joints
Links:
- link baseLink: geometry collision mesh filename=/Objects/samurai_monastry.obj scale=0.4 0.4 0.48; visual mesh filename=/Objects/samurai_monastry.obj scale=0.4 0.4 0.4
